File: AC DC converter LM317/AC DC converter LM317.kicad_pcb (KiCad board)
At the start: 2 copper layers, 50 x 50 mm, 0 parts

Commit message: Finished PCB and Schematic
Parts:
- added C1: 1000uF, Capacitor_THT:CP_Radial_D10.0mm_P5.00mm, F.Cu at (110.4, 101.0)
- added C2: 100nF, Capacitor_THT:C_Rect_L7.0mm_W2.5mm_P5.00mm, F.Cu at (113.0, 110.0)
- added C3: 100nF, Capacitor_THT:C_Rect_L7.0mm_W2.5mm_P5.00mm, F.Cu at (116.0, 110.0)
- added C4: 1000uF, Capacitor_THT:CP_Radial_D10.0mm_P5.00mm, F.Cu at (140.0, 101.0)
- added D1: 1N4007, Diode_THT:D_DO-41_SOD81_P10.16mm_Horizontal, F.Cu at (134.6, 93.6)
- added D2: 1N4007, Diode_THT:D_DO-41_SOD81_P10.16mm_Horizontal, F.Cu at (127.4, 105.6)
- added D3: 1N4007, Diode_THT:D_DO-41_SOD81_P10.16mm_Horizontal, F.Cu at (115.4, 93.6)
- added D4: 1N4007, Diode_THT:D_DO-41_SOD81_P10.16mm_Horizontal, F.Cu at (122.6, 105.6)
- added Fuse: Fuse 5x20mm, Fuse:Fuseholder_Cylinder-5x20mm_Stelvio-Kontek_PTF78_Horizontal_Open, F.Cu at (113.7, 78.5)
- added H1: MountingHole_Pad, MountingHole:MountingHole_3.2mm_M3_Pad, F.Cu at (104.0, 75.0)
- added H2: MountingHole_Pad, MountingHole:MountingHole_3.2mm_M3_Pad, F.Cu at (146.0, 75.0)
- added H3: MountingHole_Pad, MountingHole:MountingHole_3.2mm_M3_Pad, F.Cu at (104.0, 117.0)
- added H4: MountingHole_Pad, MountingHole:MountingHole_3.2mm_M3_Pad, F.Cu at (146.0, 117.0)
- added J1: Input AC, TerminalBlock:TerminalBlock_bornier-2_P5.08mm, F.Cu at (107.0, 82.5)
- added J2: Output, TerminalBlock:TerminalBlock_bornier-2_P5.08mm, F.Cu at (143.0, 87.0)
- added J3: Conn_01x04_Socket, Connector_PinHeader_2.54mm:PinHeader_1x04_P2.54mm_Vertical, F.Cu at (136.3, 116.5)
- added J4: Conn_01x02_Pin, Connector_PinHeader_2.54mm:PinHeader_1x02_P2.54mm_Vertical, F.Cu at (146.0, 91.6)
- added R1: 240, Resistor_THT:R_Axial_DIN0207_L6.3mm_D2.5mm_P7.62mm_Horizontal, F.Cu at (125.2, 109.0)
- added R2: 510, Resistor_THT:R_Axial_DIN0207_L6.3mm_D2.5mm_P7.62mm_Horizontal, F.Cu at (125.2, 112.5)
- added R3: 220, Resistor_THT:R_Axial_DIN0207_L6.3mm_D2.5mm_P7.62mm_Horizontal, F.Cu at (136.0, 112.3)
- added RV1: 10k, Potentiometer_THT:Potentiometer_Bourns_3296W_Vertical, F.Cu at (140.9, 110.0)
- added U1: LM317_TO-220, Package_TO_SOT_THT:TO-220-3_Vertical, F.Cu at (118.1, 117.0)
Routing:
- net VOUT: track 0.00 -> 54.1 mm
- net VIN 15V DC: track 0.00 -> 35.8 mm
- net Net-(D1-K): track 0.00 -> 20.1 mm
- net Net-(J3-Pin_4): track 0.00 -> 15.5 mm
- net Net-(D3-K): track 0.00 -> 15.3 mm
- net Net-(J3-Pin_3): track 0.00 -> 15.0 mm
- net Net-(J3-Pin_1): track 0.00 -> 12.2 mm
- net Net-(J1-Pin_1): track 0.00 -> 9.13 mm
- net Net-(R2-Pad2): track 0.00 -> 3.39 mm
- net GND: track 0.00 -> 0.06 mm, vias 0 -> 36
- added copper zone on B.Cu, net GND
- added copper zone on F.Cu, net GND
Other:
- outline, holes or cut-outs redrawn
- board text added: "+"
- board text added: "-"
- board text added: "AC-DC Converter Circuit"
- board text added: "AC-DC Converter Circuit by Gilbert"
- board text added: "Adjustable"
- board text added: "Fixed 5V"
- board text added: "Hi, what you're looking for?"
- board text added: "INPUT AC 0-24V"
- board text added: "Keep calm and let the flux flow"
- board text added: "OUTPUT DC"
- board text added: "Version_1.0_121025"
- board text added: "Voltmeter"
